File: pcb/dropkick.kicad_pcb (KiCad board)
At the start: 2 copper layers, 44.5 x 50.8 mm, 54 parts, among them J1 Conn_01x08, SW1 450405020524, SW2 KMR211NG_LFS, U1 ATSAMD21G18A-AUT, U2 QFN_M8C-0_UBL, U3 MCP73831T-2ACI/OT, U4 DPS310XTSA1, U5 MPU-6050, U6 SPX3819-3.3, X1 microUSB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

Commit message: Reorganize footprint libraries
Parts:
- B1: footprint lib_fr:CR1220-2 -> lib_fp:CR1220-2
- C1, C10, C12, C13, C5, C6, C7, C8, R1, R10, R14, R2, R3, R6, R7, R8, R9, SJ4: footprint lib_fr:0603-NO -> lib_fp:0603-NO
- C11, C2, C3, C4, C9: footprint lib_fr:0805-NO -> lib_fp:0805-NO
- CHG1, L1, L2: footprint lib_fr:CHIPLED_0805_NOOUTLINE -> lib_fp:CHIPLED_0805_NOOUTLINE
- D1: footprint lib_fr:SOD-123 -> lib_fp:SOD-123
- D2: footprint lib_fr:CHIPLED_0603_NOOUTLINE -> lib_fp:CHIPLED_0603_NOOUTLINE
- H1, H2, H3, H4: footprint lib_fr:MOUNTINGHOLE_2.5_PLATED -> lib_fp:MOUNTINGHOLE_2.5_PLATED
- J1: footprint Connector_PinHeader_2.54mm:PinHeader_1x08_P2.54mm_Vertical -> lib_fp:PinHeader_1x08_P2.54mm_Vertical
- JP2: footprint lib_fr:3221-10-0300-00-TR -> lib_fp:3221-10-0300-00-TR
- R11, R12, R4, R5: footprint Resistor_SMD:R_0603_1608Metric -> lib_fp:R_0603_1608Metric
- REF**: footprint Symbol:OSHW-Logo2_14.6x12mm_SilkScreen -> lib_fp:OSHW-Logo2_14.6x12mm_SilkScreen
- SW1: footprint lib_fr:450405020524 -> lib_fp:450405020524
- SW2: footprint lib_fr:KMR211NG LFS -> lib_fp:KMR211NG LFS
- TP1: footprint lib_fr:TESTPOINT_ROUND_1.5MM -> lib_fp:TESTPOINT_ROUND_1.5MM
- U1: footprint lib_fr:ATSAMD21G15B-AU -> lib_fp:ATSAMD21G15B-AU
- U2: footprint lib_fr:CAM-M8C-0 -> lib_fp:CAM-M8C-0
- U3, U6: footprint lib_fr:SOT23-5 -> lib_fp:SOT23-5
- U4: footprint lib_fr:DPS310XTSA1 -> lib_fp:DPS310XTSA1
- U5: footprint lib_fr:QFN24_4MM_SMSC -> lib_fp:QFN24_4MM_SMSC
- X1: footprint lib_fr:4UCONN_20329_V2 -> lib_fp:4UCONN_20329_V2
- X2: footprint lib_fr:JSTPH2 -> lib_fp:JSTPH2
- X3: footprint lib_fr:MICROSD -> lib_fp:MICROSD
- X4: footprint lib_fr:U.FL -> lib_fp:U.FL
- X5: footprint lib_fr:XTAL3215 -> lib_fp:XTAL3215

Commit message: Add BOM, minor footprint fixes
Parts:
- added REF**: OSHW-Logo2_14.6x12mm_SilkScreen, lib_fp:OSHW-Logo2_14.6x12mm_SilkScreen, F.Cu at (99.2, 80.3)
Other:
- board text added: "Dropkick V3 Riley Rainey"

Commit message: V4 board candidate
Parts:
- removed the REF** at (99.2, 80.3)
- added R13: 200, Resistor_SMD:R_0603_1608Metric, F.Cu at (95.9, 82.7)
- added R15: 200, Resistor_SMD:R_0603_1608Metric, F.Cu at (96.0, 81.1)
- added REF**: OSHW-Logo2_7.3x6mm_SilkScreen, Symbol:OSHW-Logo2_7.3x6mm_SilkScreen, F.Cu at (86.7, 76.6)
- C1, C10, C5: value 1uF -> 1µF
- C11, C2: value 10uF -> 10µF
- C12, C6: value 0.1uF -> 0.1µF
- CHG1: value ORANGE -> ORANGE LED
- D2, L1: value GREEN -> GREEN LED
- J1: value Conn_01x08 -> Conn_01x10; footprint lib_fp:PinHeader_1x08_P2.54mm_Vertical -> Connector_PinSocket_2.54mm:PinSocket_1x10_P2.54mm_Vertical
- L2: value RED -> RED LED
- R1, R3: value 100k -> 100K
- U1: value ATSAMD21G18A-AUT -> ATSAMD21G18A-AUT
- U2: value QFN_M8C-0_UBL -> CAM-M8C-0
- X1: value microUSB -> USB micro-B
- moved REF** 5.26 mm to (90.9, 68.5)
- moved R12 0.22 mm to (103.0, 68.9)
- moved J1 0.13 mm to (105.6, 60.8)
Connections:
- J1 pad 2: /SCL -> +3V3
- J1 pad 3: /SDA -> /SCL
- J1 pad 4: GND -> /SDA
- J1 pad 5: /AREF -> GND
- J1 pad 6: /A0 -> /AREF
- J1 pad 7: /A1 -> /A0
- J1 pad 8: /D0 -> /A1
- U1 pad 37: /RX -> unconnected-(U1-Pad37)
- U1 pad 38: /TX -> unconnected-(U1-Pad38)
- U2 pad 25: unconnected-(U2-Pad25) -> Net-(R13-Pad2)
- U2 pad 26: unconnected-(U2-Pad26) -> Net-(R15-Pad2)
Routing:
- net /D1: track 0.00 -> 29.4 mm, vias 0 -> 2
- net /D0: track 23.1 -> 33.7 mm, vias 1 -> 2
- net /SCL: track 76.3 -> 71.9 mm, vias 2 -> 3
- net +3V3: track 161.6 -> 157.3 mm
- net Net-(R15-Pad2): track 0.00 -> 4.18 mm
- net Net-(R13-Pad2): track 0.00 -> 4.01 mm
- net /D13: track 34.5 -> 37.9 mm
- net /A1: track 24.7 -> 26.4 mm
- net /SDA: track 71.6 -> 70.5 mm, vias 3 -> 4
- net /AREF: track 26.9 -> 27.8 mm
- net /A0: track 22.1 -> 23.0 mm
Other:
- board text added: "+3.3V"
- board text added: "D1"
- board text added: "Dropkick V4 Copyright (c) 2022 Riley Rainey https://GitHub.com/rrainey/dropkick/"
- board text added: "Dropkick V4 Riley Rainey"
- board text removed: "Dropkick V3 Copyright (c) 2022 Riley Rainey https://GitHub.com/rrainey/dropkick/"
- board text removed: "Dropkick V3 Riley Rainey"
