File: pcb/dropkick.kicad_sch (KiCad schematic)
At the start: 50 parts, among them SW1 450405020524, SW2 KMR211NG_LFS, U1 ATSAMD21G18A-AUT, U2 SAM-M8Q-0-10, U3 MCP73831T-2ACI/OT, U4 DPS310XTSA1, U5 MPU-6050, U6 SPX3819-3.3, X1 microUSB, X2 JSTPH, X3 microsd, X5 32768Hz

Commit message: V2-SAM working draft
Parts:
- removed C5: 1uF, Capacitor_SMD:C_0603_1608Metric, symbol Adafruit Feather M0 Adalogger-eagle-import:CAP_CERAMIC0603_NO
- removed JP4: HEADER-1X12, 1X12_ROUND, symbol Adafruit Feather M0 Adalogger-eagle-import:HEADER-1X12
- removed JP5: HEADER-1X16ROUND, 1X16_ROUND, symbol Adafruit Feather M0 Adalogger-eagle-import:HEADER-1X16ROUND
- removed R11: 4.7K, RESPACK_4X0603, symbol Adafruit MPU6050-eagle-import:RESISTOR_4PACK
- removed R14: 10K, Resistor_SMD:R_0603_1608Metric, symbol Adafruit MPU6050-eagle-import:RESISTOR_0603_NOOUT
- removed SJ4: SOLDERJUMPER, 310:0603-NO, symbol Adafruit MPU6050-eagle-import:SOLDERJUMPER
- removed TP1: TESTPOINTROUND1.5MM, TESTPOINT_ROUND_1.5MM, symbol Adafruit Ultimate GPS FeatherWing-eagle-import:TESTPOINTROUND1.5MM
- added J1: Conn_01x08, Connector_PinHeader_2.54mm:PinHeader_1x09_P2.54mm_Vertical, symbol Connector_Generic:Conn_01x09
- added R10, R9: 10K, Resistor_SMD:R_0603_1608Metric, symbol Adafruit MPU6050-eagle-import:RESISTOR_0603_NOOUT
- CHG1, L1, L2: footprint CHIPLED_0805_NOOUTLINE -> lib_fr:CHIPLED_0603_NOOUTLINE; symbol Adafruit Feather M0 Adalogger-eagle-import:LED0805_NOOUTLINE -> Adafruit Feather M0 Adalogger-eagle-import:LED0603
- D2: footprint CHIPLED_0603_NOOUTLINE -> lib_fr:CHIPLED_0603_NOOUTLINE
- H1, H2, H3, H4: footprint logger:MOUNTINGHOLE_2.5_PLATED -> lib_fr:MOUNTINGHOLE_2.5_PLATED
- JP1: renamed from JP2; footprint logger:3221-10-0300-00-TR -> lib_fr:3221-10-0300-00-TR
- SW1: footprint logger:450405020524 -> lib_fr:450405020524
- SW2: footprint logger:KMR211NG LFS -> lib_fr:KMR211NG LFS
- U4: renamed from U1; footprint logger:ATSAMD21G15B-AU -> lib_fr:ATSAMD21G15B-AU
- U5: renamed from U4; footprint logger:DPS310XTSA1 -> lib_fr:DPS310XTSA1
- renumbered C6 to C10, C12 to C11, C13 to C12, C11 to C5, C7 to C6, C8 to C7, C9 to C8, C10 to C9, R3 to R2, R2 to R3, R6 to R4, R7 to R5, R8 to R6, R9 to R7, R10 to R8, U6 to U1, U5 to U6, X5 to X4
Connections:
- net 3.3V is gone; now on net +3V3: C10.1, C5.1, R8.1, U2.17 (VCC), U2.2 (VCC_IO), U5.6 (VDDIO), U5.8 (VDD), U6.13 (VDD), U6.8 (VLOGIC)
- net VCC is gone; now on net +3V3: JP1.1
- net +3V3: now also J1.2 (Pin_2), R10.1, R9.1
- net A0: now also J1.6 (Pin_6)
- net AREF: now also J1.5 (Pin_5)
- net D0: now also J1.7 (Pin_7)
- net D1: now also J1.8 (Pin_8)
- net GND: now also J1.9 (Pin_9)
- net SCL: now also J1.3 (Pin_3), R9.2
- net SDA: now also J1.4 (Pin_4), R10.2
- net VBAT: now also J1.1 (Pin_1)
- no-connect marks 21 -> 23
Other:
- note removed: "N/C"
- note removed: "RXD"
- note removed: "RXLED"
- note removed: "TXD"
- note removed: "TXLED"
- note removed: "USBHOSTEN"
- moved on the sheet: B1, C10, C11, C12, C5, U2, U5, U6

Commit message: test of 4-layer PCB
Connections:
- net GND: no longer U4.EPAD (GND)
Changed lines of the file:
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@@
     (pin "8")
     (pin "9")
-    (pin "EPAD")
   )
   (symbol (lib_id "Adafruit Feather M0 Adalogger-eagle-import:GND") (at 22.86 59.69 0) (unit 1)
