File: pcb-sam/dropkick.kicad_pcb (KiCad board)
At the start: 2 copper layers, 44.5 x 50.8 mm, 48 parts, among them J1 Conn_01x08, SW1 450405020524, SW2 KMR211NG_LFS, U1 SPX3819-3.3, U2 SAM-M8Q-0-10, U3 MCP73831T-2ACI/OT, U4 ATSAMD21G18A-AUT, U5 DPS310XTSA1, U6 MPU-6050, X1 microUSB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

Commit message: V3-SAM gerber files
Parts:
- U2: footprint lib_fr:MODULE_SAM-M8Q-0-10 -> lib_fr:MODULE_SAM-M8Q-0-10_large
