File: pcb-sam/dropkick.kicad_sch (KiCad schematic)
At the start: 46 parts, among them J1 Conn_01x08, SW1 450405020524, SW2 KMR211NG_LFS, U1 SPX3819-3.3, U2 SAM-M8Q-0-10, U3 MCP73831T-2ACI/OT, U4 ATSAMD21G18A-AUT, U5 DPS310XTSA1, U6 MPU-6050, X1 microUSB, X2 JSTPH, X3 microsd, X4 32768Hz

Commit message: v3 SAM PCB
Parts:
- removed X1: microUSB, 4UCONN_20329_V2, symbol Adafruit Feather M0 Adalogger-eagle-import:USB_MICRO_20329_V2
- added C13: 10nF, Capacitor_SMD:C_0603_1608Metric, symbol Adafruit MPU6050-eagle-import:CAP_CERAMIC0603_NO
- added J2: USB C USB2.0, Connector_USB:USB_C_Receptacle_GCT_USB4085, symbol Connector:USB_C_Receptacle_USB2.0
- added R11, R12: 5.1K, Resistor_SMD:R_0402_1005Metric, symbol Adafruit DPS310-eagle-import:RESISTOR_0603
- B1: MANUFACTURER (none) -> Keystone; MPN (none) -> 1056TR
- C11, C12: footprint 0603-NO -> Capacitor_SMD:C_0603_1608Metric
- CHG1: value AMBER -> LTST-C191KFKT; MANUFACTURER (none) -> Lite-On; MPN (none) -> LTST-C191KFKT
- D2: value GRN -> LTST-S270KGKT; MPN (none) -> LTST-S270KGKT
- JP1: MPN (none) -> 3221-10-0300-00-TR
- L1: value GRN -> LTST-S270KGKT; MANUFACTURER (none) -> Lite-On; MPN (none) -> LTST-S270KGKT
- L2: value RED -> LTST-S270KRKT; MANUFACTURER (none) -> Lite-On; MPN (none) -> LTST-S270KRKT
- R1, R2, R3: footprint 0603-NO -> Resistor_SMD:R_0603_1608Metric
- SW1: MANUFACTURER (none) -> Wurth; MPN (none) -> 450405020524
- SW2: MPN (none) -> KMR211NG_LFS
- U1: MPN (none) -> SPX3819-3.3
- U2: MPN (none) -> SAM-M8Q-0-10
- U3: MPN (none) -> MCP73831T-2ACI/OT
- U4: value ATSAMD21G18A-AUT -> ATSAMD21G18A-AUT; MPN (none) -> ATSAMD21G18A-AUT
- U5: MANUFACTURER (none) -> Infineon; MPN (none) -> DPS310XTSA1
- X2: MANUFACTURER (none) -> JST
- X3: value microsd -> MEM2061-01-188-00-A; MANUFACTURER (none) -> GCT; MPN (none) -> MEM2061-01-188-00-A
Connections:
- net INT is gone; now on net D11: U6.12 (INT)
- net +3V3: now also C13.1; no longer U6.8 (VLOGIC)
- net D+: now also J2.A6 (D+), J2.B6 (D+)
- net D-: now also J2.A7 (D-), J2.B7 (D-)
- net GND: now also J2.A1 (GND), J2.A12 (GND), J2.B1 (GND), J2.B12 (GND), R11.2, R12.2
- net VBUS: now also J2.A4 (VBUS), J2.A9 (VBUS), J2.B4 (VBUS), J2.B9 (VBUS)
- new net: J2.B5 (CC2), R12.1
- new net: C13.2, U6.8 (VLOGIC)
- new net: J2.A5 (CC1), R11.1
- no-connect marks 23 -> 25
Other:
- moved on the sheet: H1, H2, H3, H4, R1, R3

Commit message: V4 SAM PCB
Parts:
- removed C10, C11: 0.1uF, Capacitor_SMD:C_0603_1608Metric, symbol Adafruit MPU6050-eagle-import:CAP_CERAMIC0603_NO
- removed C12: 2.2nF, Capacitor_SMD:C_0603_1608Metric, symbol Adafruit MPU6050-eagle-import:CAP_CERAMIC0603_NO
- removed C13: 10nF, Capacitor_SMD:C_0603_1608Metric, symbol Adafruit MPU6050-eagle-import:CAP_CERAMIC0603_NO
- removed H4: MountingHole, lib_fr:MOUNTINGHOLE_2.5_PLATED, symbol Mechanical:MountingHole
- removed U5: DPS310XTSA1, lib_fr:DPS310XTSA1, symbol dropkick:DPS310XTSA1
- removed U6: MPU-6050, QFN24_4MM_SMSC, symbol Adafruit MPU6050-eagle-import:MPU-6050
- added C10: 0.1uF, Capacitor_SMD:C_0603_1608Metric, symbol Device:C_Small
- added C11: 2.2uF, Capacitor_SMD:C_0603_1608Metric, symbol Device:C_Small
- added C12, C13: 100nF, Capacitor_SMD:C_0603_1608Metric, symbol Device:C_Small
- added C14: 10nF, Capacitor_SMD:C_0603_1608Metric, symbol Device:C_Small
- added U5: BMP390, lib_fr:LGA10_BMP390_BOS, symbol dropkick:BMP390
- added U6: ICM-42688-P, lib_fr:PQFN50P300X250X97-14N, symbol dropkick:ICM-42688-P
- C1, C2, C3, C4, C5, C6, C9: NOTES (none) -> X7R
- C7, C8: NOTES (none) -> MLCC - SMD/SMT 50V 22pF C0G 0603 1%
- CHG1: NOTES (none) -> YELLOW LED
- D1: value MBR120 -> SCHOTTKY 20V; footprint SOD-123 -> Diode_SMD:D_SOD-123F; MPN (none) -> SM5817PL-TP; NOTES (none) -> 20V 1A Substitutions OK
- J1: renamed from J2; value USB C USB2.0 -> USB-C 2.0
- J2: renamed from X2; value JSTPH -> BATT; footprint JSTPH2 -> lib_fr:JSTPH2; MPN (none) -> S2B-PH-SM4-TB
- L1: NOTES (none) -> GREEN LED
- L2: NOTES (none) -> RED LED
- L3: renamed from D2; NOTES (none) -> GREEN LED
- R1: renamed from R11; NOTES (none) -> 1%
- R10: renamed from R8; value 10K -> 2.2K; NOTES (none) -> 1%
- R11: renamed from R9; NOTES (none) -> 1%
- R12: renamed from R10; NOTES (none) -> 1%
- R2: renamed from R12; NOTES (none) -> 1%
- R3: renamed from R1; NOTES (none) -> 1%
- R4: renamed from R2; NOTES (none) -> 1%
- R5: renamed from R3; NOTES (none) -> 1%
- R6: renamed from R4; NOTES (none) -> 1%
- R7: renamed from R5; NOTES (none) -> 1%
- R8: renamed from R6; NOTES (none) -> 1%
- R9: renamed from R7; value 1K -> 2.2K; NOTES (none) -> 1%
- SW2: MANUFACTURER (none) -> C&K
- U2: value SAM-M8Q-0-10 -> SAM-M10Q; MANUFACTURER ublox -> u-blox; MPN SAM-M8Q-0-10 -> SAM-M10Q-00B
- U4: MANUFACTURER (none) -> Microchip
- X2: renamed from X4; MANUFACTURER (none) -> SEIKO EPSON; MPN (none) -> FC-135 32.7680KA-A5; NOTES (none) -> MINI SMD XTL KHZ (3.3x1.5mm)+/-20PPM,-40-85C 12.5PF 3K TR
- renumbered J1 to J3, JP1 to J4, X3 to X1
Connections:
- net +3V3: now also C10.1, C11.1, C12.1, C13.1, C14.1, U5.1 (VDDIO), U5.10 (VDD), U5.6 (CSB), U6.12 (AP_CS), U6.5 (VDDIO), U6.8 (VDD)
- net D11: now also U6.4 (INT1/INT)
- net D12: now also U6.9 (INT2/FSYNC/CLKIN)
- net D6: now also U5.7 (INT)
- net D8: now also R9.1; no longer L1.A
- net GND: now also L1.C, C10.2, C11.2, C12.2, C13.2, C14.2, U5.3 (VSS), U5.5 (SDO), U5.8 (VSS), U5.9 (VSS), U6.1 (AP_SDO/AP_AD0), U6.11 (RESV_11), U6.6 (GND), U6.7 (RESV_7); no longer R9.2
- net SCL: now also U5.2 (SCK), U6.13 (AP_SCL/AP_SCLK)
- net SDA: now also U5.4 (SDI), U6.14 (AP_SDA/AP_SDIO/AP_SDI)
- net VBAT: now also D1.2; no longer D1.A
- net VBUS: now also D1.1; no longer D1.C
- new net: L1.A, R9.2
- no-connect marks 25 -> 26
Other:
- note added: "3.7V Li-Poly Battery"
- note added: "DNP"
- note removed: ""ON" LED"
- moved on the sheet: C6, C7, C8, C9, CHG1, H1, H2, H3, J3, J4, L1, L2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

Commit message: V4 SAM
Parts:
- B1: NOTES (none) -> BATT HOLDER
- J1: NOTES (none) -> USB-C
- J2: NOTES (none) -> 2 PIN RECEPTACLE
- J3: MPN (none) -> DNP
- U1: NOTES (none) -> IC REG LINEAR 3.3V 500MA
- U2: NOTES (none) -> GNSS RECEIVER
- U3: NOTES (none) -> IC BATT CNTL LI-ION 1CEL
- U4: NOTES (none) -> 32 BIT MCU 256K FLASH
Connections:
- no-connect marks 26 -> 36
Other:
- note added: "DO NOT PLACE"
- note added: "NOT CONNECTED"
- note added: "POWER DESIGNATORS"
- note removed: "DNP"
- moved on the sheet: C8, CHG1, H1, H2, H3, J4, R11, R12, R6, R7, U3
